File: precision-clock-pcb/gps.kicad_sch (KiCad schematic)
At the start: 1 part, among them U5 PA1616S

Commit message: schematic work done
Parts:
- added C27: 0.1uF, symbol Device:C
- added D5: LED, symbol Device:LED
- added J2: ANT, Connector_Coaxial:MMCX_Molex_73415-1471_Vertical, symbol Connector:Conn_Coaxial
- added R42: 1K, symbol Device:R
Connections:
- net +3V3: now reaches U5.1 (VCC)
- net +3V3: now also C27.1
- net RX: now reaches U5.10 (RX0)
- net at U5.11 (EXT_ANT): now also J2.1 (In)
- net GND: now reaches U5.12 (GND), U5.19 (GND), U5.3 (GND), U5.8 (GND)
- net GND: now also C27.2, J2.2 (Ext), R42.1
- net PPS: now reaches U5.13 (1PPS)
- net at U5.5 (3D-FIX): now also D5.2 (A)
- net TX: now reaches U5.9 (TX0)
- new net: D5.1 (K), R42.2

Commit message: board work
Parts:
- C26: renamed from C27; value 0.1uF -> 100nF; footprint (none) -> Capacitor_SMD:C_0402_1005Metric
- D1: renamed from D5; footprint (none) -> LED_SMD:LED_0603_1608Metric
- R21: renamed from R42; footprint (none) -> Resistor_SMD:R_0402_1005Metric
- renumbered J2 to J3
Changed lines of the file:
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@@
 		(dnp no)
 		(fields_autoplaced yes)
-		(property "Reference" "#PWR039"
+		(property "Reference" "#PWR042"
 			(at 135.89 99.06 0)
 			(effects
@@
 			(project ""
 				(path "/3cbd0e8e-3ba4-43b1-82ac-749e7a469b5f/91dee3c8-a62e-4987-889d-37e8aa06db65"
-					(reference "#PWR039")
+					(reference "#PWR042")
 					(unit 1)
 				)
@@
 		(dnp no)
 		(fields_autoplaced yes)
-		(property "Reference" "J2"
+		(property "Reference" "J3"
 			(at 86.6774 78.74 0)
 			(effects
@@
 			(project ""
 				(path "/3cbd0e8e-3ba4-43b1-82ac-749e7a469b5f/91dee3c8-a62e-4987-889d-37e8aa06db65"
-					(reference "J2")
+					(reference "J3")
 					(unit 1)
 				)
@@
 		(dnp no)
 		(fields_autoplaced yes)
-		(property "Reference" "D5"
+		(property "Reference" "D1"
 			(at 107.6325 73.66 0)
 			(effects
@@
 			)
 		)
-		(property "Footprint" ""
+		(property "Footprint" "LED_SMD:LED_0603_1608Metric"
 			(at 109.22 80.01 0)
 			(effects
@@
 			(project ""
 				(path "/3cbd0e8e-3ba4-43b1-82ac-749e7a469b5f/91dee3c8-a62e-4987-889d-37e8aa06db65"
-					(reference "D5")
+					(reference "D1")
 					(unit 1)
 				)
@@
 		(on_board yes)
 		(dnp no)
-		(property "Reference" "R42"
+		(property "Reference" "R21"
 			(at 101.6 77.724 90)
 			(effects
@@
 			)
 		)
-		(property "Footprint" ""
+		(property "Footprint" "Resistor_SMD:R_0402_1005Metric"
 			(at 101.6 81.788 90)
 			(effects
@@
 			(project ""
 				(path "/3cbd0e8e-3ba4-43b1-82ac-749e7a469b5f/91dee3c8-a62e-4987-889d-37e8aa06db65"
-					(reference "R42")
+					(reference "R21")
 					(unit 1)
 				)
@@
 		(dnp no)
 		(fields_autoplaced yes)
-		(property "Reference" "C27"
+		(property "Reference" "C26"
 			(at 106.68 60.9599 0)
 			(effects
@@
 			)
 		)
-		(property "Value" "0.1uF"
+		(property "Value" "100nF"
 			(at 106.68 63.4999 0)
 			(effects
@@
 			)
 		)
-		(property "Footprint" ""
+		(property "Footprint" "Capacitor_SMD:C_0402_1005Metric"
 			(at 103.8352 66.04 0)
 			(effects
@@
 			(project ""
 				(path "/3cbd0e8e-3ba4-43b1-82ac-749e7a469b5f/91dee3c8-a62e-4987-889d-37e8aa06db65"
-					(reference "C27")
+					(reference "C26")
 					(unit 1)
 				)
@@
 		(on_board yes)
 		(dnp no)
-		(property "Reference" "#PWR042"
+		(property "Reference" "#PWR039"
 			(at 97.79 86.36 0)
 			(effects
@@
 			(project "precision-clock"
 				(path "/3cbd0e8e-3ba4-43b1-82ac-749e7a469b5f/91dee3c8-a62e-4987-889d-37e8aa06db65"
-					(reference "#PWR042")
+					(reference "#PWR039")
 					(unit 1)
 				)
@@
 		(dnp no)
 		(fields_autoplaced yes)
-		(property "Reference" "#PWR043"
+		(property "Reference" "#PWR038"
 			(at 86.36 96.52 0)
 			(effects
@@
 			(project "precision-clock"
 				(path "/3cbd0e8e-3ba4-43b1-82ac-749e7a469b5f/91dee3c8-a62e-4987-889d-37e8aa06db65"
-					(reference "#PWR043")
-					(unit 1)
-				)
+					(reference "#PWR038")
+					(unit 1)
+				)

Commit message: Board Rev 1.0 Release
Connections:
- net ANT: now reaches J3.1 (In), U5.11 (EXT_ANT)
Changed lines of the file:
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@@
+		)
+	)
+	(label "ANT"
+		(at 102.87 85.09 0)
+		(effects
+			(font
+				(size 1.27 1.27)
+			)
+			(justify left bottom)
 		)
 	)

Commit message: BOM, CSV, and STEP exports
Parts:
- C26: JLCPCB PN (none) -> C77014; MFR PN (none) -> GRM155R71E104KE14D
- D1: JLCPCB PN (none) -> C3030991; MFR PN (none) -> 150060RS75000
- J3: JLCPCB PN (none) -> C588477; MFR PN (none) -> 0734151471
- R21: JLCPCB PN (none) -> C106235; MFR PN (none) -> RC0402FR-071KL
- U5: MFR PN (none) -> PA1616S
Changed lines of the file:
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@@
+			)
+		)
+		(property "JLCPCB PN" "C588477 "
+			(at 86.36 85.09 0)
+			(effects
+				(font
+					(size 1.27 1.27)
+				)
+				(hide yes)
+			)
+		)
+		(property "MFR PN" "0734151471"
+			(at 86.36 85.09 0)
+			(effects
+				(font
+					(size 1.27 1.27)
+				)
+				(hide yes)
 			)
 		)
@@
 			)
 		)
+		(property "JLCPCB PN" "C3030991 "
+			(at 109.22 80.01 0)
+			(effects
+				(font
+					(size 1.27 1.27)
+				)
+				(hide yes)
+			)
+		)
+		(property "MFR PN" "150060RS75000"
+			(at 109.22 80.01 0)
+			(effects
+				(font
+					(size 1.27 1.27)
+				)
+				(hide yes)
+			)
+		)
 		(pin "1"
 		)
@@
 			)
 		)
+		(property "JLCPCB PN" "C106235 "
+			(at 101.6 80.01 90)
+			(effects
+				(font
+					(size 1.27 1.27)
+				)
+				(hide yes)
+			)
+		)
+		(property "MFR PN" "RC0402FR-071KL"
+			(at 101.6 80.01 90)
+			(effects
+				(font
+					(size 1.27 1.27)
+				)
+				(hide yes)
+			)
+		)
 		(pin "2"
 		)
@@
 			)
 		)
+		(property "JLCPCB PN" ""
+			(at 135.89 74.93 0)
+			(effects
+				(font
+					(size 1.27 1.27)
+				)
+				(hide yes)
+			)
+		)
+		(property "MFR PN" "PA1616S"
+			(at 135.89 74.93 0)
+			(effects
+				(font
+					(size 1.27 1.27)
+				)
+				(hide yes)
+			)
+		)
 		(pin "15"
 		)
@@
 			(at 102.87 62.23 0)
 			(effects
+				(font
+					(size 1.27 1.27)
+				)
+				(hide yes)
+			)
+		)
+		(property "JLCPCB PN" "C77014"
+			(at 102.87 62.23 0)
+			(effects
+				(font
+					(size 1.27 1.27)
+				)
+				(hide yes)
+			)
+		)
+		(property "MFR PN" "GRM155R71E104KE14D"
+			(at 102.87 62.23 0)
+			(effects
