File: precision-clock-pcb/precision-clock.kicad_pcb (KiCad board)
At the start: 4 copper layers, 150 parts, among them J1 USB_C_Receptacle_USB2.0_14P, J2 TC2050, J3 ANT, Q1 SFH320, Q10 BSS138, Q11 BSS138, Q12 BSS138, Q13 BSS138, Q14 BSS138, Q15 BSS138, Q16 BSS138, Q2 SFH320, Q3 BSS138, Q4 BSS83P, Q5 BSS138, Q6 BSS138, Q7 BSS138, Q8 BSS138, Q9 BSS138, SW1 BUTTON, SW2 BUTTON, SW3 BOOTSEL, SW4 RESET, U1 W25Q128JVS, U10 SN74ABT244ADW, U2 USBLC6-2P6, U3 NCP1117-3.3_SOT223, U4 RP2350_80QFN, U5 PA1616S, U6 DS3232M, U7 CD74HCT238M96, U8 CD74HCT238M96, U9 SN74ABT244ADW, Y1 ABM8-272-T3

Commit message: board work
Parts:
- BT1, C26, C28, C29, C30, D1, J1, J2, L1, Q15, Q16, Q5, R21, R26, R27, R50, TP1, U2, U4, U5, U6, U7, Y1: moved to B.Cu
- C1: renamed from C4; moved to B.Cu
- C10: renamed from C20; moved to B.Cu
- C11: renamed from C21; moved to B.Cu
- C12: renamed from C22; moved to B.Cu
- C13: renamed from C23; moved to B.Cu
- C14: renamed from C24; moved to B.Cu
- C15: renamed from C25; moved to B.Cu
- C16: renamed from C3; moved to B.Cu
- C17: renamed from C13; moved to B.Cu
- C18: renamed from C7; moved to B.Cu
- C19: renamed from C10; moved to B.Cu
- C2: renamed from C6; moved to B.Cu
- C20: renamed from C1; moved to B.Cu
- C21: renamed from C2; moved to B.Cu
- C3: renamed from C12; moved to B.Cu
- C31: renamed from C32; moved to B.Cu
- C32: renamed from C33; moved to B.Cu
- C33: renamed from C31; moved to B.Cu
- C4: renamed from C14; moved to B.Cu
- C5: renamed from C15; moved to B.Cu
- C6: renamed from C16; moved to B.Cu
- C7: renamed from C17; moved to B.Cu
- C8: renamed from C18; moved to B.Cu
- C9: renamed from C19; moved to B.Cu
- Q10: renamed from Q6; moved to B.Cu
- Q11: renamed from Q7; moved to B.Cu
- Q12: renamed from Q9; moved to B.Cu
- Q13: renamed from Q11; moved to B.Cu
- Q14: renamed from Q13; moved to B.Cu
- Q3: renamed from Q4; moved to B.Cu
- Q4: renamed from Q3; moved to B.Cu
- Q6: renamed from Q8; moved to B.Cu
- Q7: renamed from Q10; moved to B.Cu
- Q8: renamed from Q12; moved to B.Cu
- Q9: renamed from Q14; moved to B.Cu
- R1: renamed from R3; moved to B.Cu
- R10: renamed from R20; moved to B.Cu
- R11: renamed from R9; moved to B.Cu
- R2: renamed from R4; moved to B.Cu
- R22: renamed from R23; moved to B.Cu
- R24: renamed from R25; moved to B.Cu
- R25: renamed from R24; moved to B.Cu
- R28: renamed from R31; moved to B.Cu
- R29: renamed from R33; moved to B.Cu
- R3: renamed from R12; moved to B.Cu
- R30: renamed from R44; moved to B.Cu
- R31: renamed from R54; moved to B.Cu
- R32: renamed from R30; moved to B.Cu
- R33: renamed from R43; moved to B.Cu
- R34: renamed from R28; moved to B.Cu
- R35: renamed from R29; moved to B.Cu
- R36: renamed from R32; moved to B.Cu
- R37: renamed from R42; moved to B.Cu
- R38: renamed from R45; moved to B.Cu
- R39: renamed from R55; moved to B.Cu
- R4: renamed from R15; moved to B.Cu
- R40: renamed from R56; moved to B.Cu
- R41: renamed from R34; moved to B.Cu
- R42: renamed from R46; moved to B.Cu
- R43: renamed from R35; moved to B.Cu
- R44: renamed from R47; moved to B.Cu
- R45: renamed from R36; moved to B.Cu
- R46: renamed from R48; moved to B.Cu
- R47: renamed from R37; moved to B.Cu
- R48: renamed from R49; moved to B.Cu
- R49: renamed from R38; moved to B.Cu
- R5: renamed from R16; moved to B.Cu
- R51: renamed from R39; moved to B.Cu
- R52: renamed from R51; moved to B.Cu
- R53: renamed from R40; moved to B.Cu
- R54: renamed from R52; moved to B.Cu
- R55: renamed from R41; moved to B.Cu
- R56: renamed from R53; moved to B.Cu
- R7: renamed from R17; moved to B.Cu
- R8: renamed from R18; moved to B.Cu
- SW1: renamed from SW3; moved to B.Cu
- SW2: renamed from SW4; moved to B.Cu
- U1: renamed from U3; moved to B.Cu
- U10: renamed from U8; moved to B.Cu
- U3: renamed from U1; moved to B.Cu
- U8: renamed from U9; moved to B.Cu
- U9: renamed from U10; moved to B.Cu
- moved Q2 505.5 mm to (510.0, 33.0), turned to 90 degrees
- moved SW4 495.2 mm to (510.1, 44.1), turned to 90 degrees
- moved SW3 491.4 mm to (510.1, 54.6), turned to 90 degrees
- moved Q16 429.1 mm to (495.0, 57.0), turned to -90 degrees
- moved Q15 404.7 mm to (471.0, 57.0), turned to -90 degrees
- moved R40 397.8 mm to (495.0, 54.5)
- moved R39 374.0 mm to (471.0, 54.5)
- moved Q14 363.6 mm to (423.0, 57.0), turned to -90 degrees
- moved D3 344.8 mm to (381.0, 38.0)
- moved D5 342.3 mm to (381.0, 52.0)
- moved R38 328.3 mm to (423.0, 54.5)
- moved Q13 320.6 mm to (381.0, 57.4), turned to 90 degrees
- moved Q12 311.0 mm to (365.0, 57.0), turned to -90 degrees
- moved R33 302.3 mm to (385.5, 37.5), turned to 90 degrees
- moved R37 290.6 mm to (381.0, 60.0), turned to 180 degrees
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- renumbered C5 to C22, C11 to C23, C8 to C24, C9 to C25, D4 to D3, D3 to D4, DS17 to DS10, DS2 to DS11, DS4 to DS12, DS7 to DS13, DS9 to DS14, DS12 to DS15, DS14 to DS16, DS16 to DS17, DS3 to DS2, DS5 to DS3, DS6 to DS4, DS8 to DS5, DS10 to DS6, DS11 to DS7, DS13 to DS8, DS15 to DS9, R13 to R12, R2 to R13, R5 to R14, R6 to R15, R7 to R16, R8 to R17, R1 to R18, R10 to R19, R11 to R20, R22 to R23, R14 to R6, R19 to R9, SW1 to SW3, SW2 to SW4
Routing:
- net /Display/SEGB1: track 0.00 -> 519.5 mm, vias 0 -> 10
- net /Display/SEGH1: track 0.00 -> 514.7 mm, vias 0 -> 10
- net /Display/SEGE1: track 0.00 -> 513.1 mm
- net /Display/SEGA1: track 0.00 -> 510.8 mm, vias 0 -> 10
- net /Display/SEGC1: track 0.00 -> 492.0 mm, vias 0 -> 9
- net /Display/SEGD1: track 0.00 -> 488.2 mm, vias 0 -> 10
- net /Display/SEGF1: track 0.00 -> 486.6 mm, vias 0 -> 9
- net /Display/SEGG1: track 0.00 -> 479.5 mm, vias 0 -> 1
- net /Display/SEGA2: track 0.00 -> 478.9 mm, vias 0 -> 10
- net /Display/SEGE2: track 0.00 -> 468.1 mm, vias 0 -> 9
- net /Display/SEGC2: track 0.00 -> 458.4 mm, vias 0 -> 10
- net /Display/SEGD2: track 0.00 -> 456.5 mm, vias 0 -> 10
- net /Display/SEGB2: track 0.00 -> 456.2 mm, vias 0 -> 1
- net /Display/SEGF2: track 0.00 -> 455.4 mm, vias 0 -> 10
- net /Display/SEGG2: track 0.00 -> 452.5 mm, vias 0 -> 9
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Other:
- board outline added: 499.5 x 34 mm

Commit message: Board Rev 1.0 Release
Parts:
- C22, C23, C24, C25, C27, J3, R12, R13, R14, R15, R16, R17, R18, R19, R20, R23, R6, R9: moved to B.Cu
- moved R20 452.3 mm to (510.0, 32.1), turned to -90 degrees
- moved C24 440.8 mm to (510.1, 57.4), turned to 180 degrees
- moved C25 438.0 mm to (510.1, 46.9), turned to 180 degrees
- moved R18 221.2 mm to (270.7, 49.0)
- moved R19 101.5 mm to (16.0, 32.0), turned to -90 degrees
- moved R9 83.4 mm to (73.5, 37.1), turned to -90 degrees
- moved R14 79.7 mm to (87.6, 47.7)
- moved R6 78.6 mm to (58.8, 42.0), turned to 180 degrees
- moved R17 78.0 mm to (71.5, 40.8), turned to 90 degrees
- moved R16 76.2 mm to (72.5, 40.8), turned to 90 degrees
- moved R13 73.5 mm to (90.5, 49.7), turned to 90 degrees
- moved R12 72.8 mm to (89.5, 49.7), turned to -90 degrees
- moved R15 70.3 mm to (87.6, 48.7)
- moved C27 58.8 mm to (80.3, 53.0), turned to -90 degrees
- moved R23 55.6 mm to (132.8, 43.2), turned to 180 degrees
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Connections:
- net Net-(J3-In) renamed /GPS/ANT
- U2 pad 5: UVBUS -> +5V
Routing:
- net /PD2: track 0.00 -> 455.1 mm, vias 0 -> 4
- net /USER_BUTTON_2: track 0.00 -> 444.0 mm, vias 0 -> 3
- net /USER_BUTTON_1: track 0.00 -> 442.6 mm, vias 0 -> 2
- net Net-(J2-Pad7): track 0.00 -> 207.9 mm, vias 0 -> 2
- net Net-(J2-Pad8): track 0.00 -> 206.2 mm, vias 0 -> 2
- net Net-(J2-Pad1): track 0.00 -> 195.7 mm, vias 0 -> 4
- net Net-(J2-Pad10): track 0.00 -> 182.7 mm, vias 0 -> 2
- net Net-(J2-Pad9): track 0.00 -> 181.8 mm, vias 0 -> 2
- net /PD1: track 0.00 -> 78.9 mm, vias 0 -> 2
- net Net-(Q6-D): track 27.2 -> 103.6 mm, vias 0 -> 2
- net Net-(Q8-D): track 27.2 -> 100.5 mm, vias 0 -> 2
- net Net-(Q9-D): track 27.2 -> 99.4 mm
- net /ADC0: track 0.00 -> 61.8 mm, vias 0 -> 2
- net Net-(Q5-D): track 27.2 -> 84.6 mm, vias 0 -> 2
- net /GPS/PPS: track 0.00 -> 57.0 mm
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- added copper zone on B.Cu, net +1V1
- added copper zone on In1.Cu, net +3V3
- added copper zone on In1.Cu, net +5V
- added copper zone on B.Cu, net GND
- added copper zone on F.Cu, net GND
- added copper zone on In2.Cu, net GND
Other:
- board size 499.5 x 34 mm -> 500 x 34 mm
- board text added: "Ordering notes: 4 layers, 1oz outer 1oz inner. Specify stackup so that In2.Cu is directly above B.Cu to ensure proper grounding of impedance controlled traces Use JLC 4 layer controlled stackup JLC041611-7628 Min via size 0.25/0.4mm, order with vias epoxy filled and capped Remove Mark and please order it in something other than Green or Yellow"
- board text added: "RP2350B Precision Clock Rev 1.0"

Commit message: BOM, CSV, and STEP exports
Other:
- board text added: "Ordering notes: Specify stackup so that In2.Cu is directly above B.Cu to ensure proper grounding of impedance controlled traces Use JLC 4 layer controlled stackup JLC04161H-7628 (default stackup) Min via size 0.25/0.4mm, order with vias epoxy filled and capped"
- board text removed: "Ordering notes: 4 layers, 1oz outer 1oz inner. Specify stackup so that In2.Cu is directly above B.Cu to ensure proper grounding of impedance controlled traces Use JLC 4 layer controlled stackup JLC041611-7628 Min via size 0.25/0.4mm, order with vias epoxy filled and capped Remove Mark and please order it in something other than Green or Yellow"
Changed lines of the file:
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@@
 	(footprint "Resistor_SMD:R_0402_1005Metric"
 		(layer "B.Cu")
-		(at 69.01 46)
+		(at 69 46)
 		(descr "Resistor SMD 0402 (1005 Metric), square (rectangular) end terminal, IPC-7351 nominal, (Body size source: IPC-SM-782 page 72, https://www.pcb-3d.com/wordpress/wp-content/uploads/ipc-sm-782a_amendment_1_and_2.pdf), generated with kicad-footprint-generator")
 		(tags "resistor")
@@
 			(size 0.6 0.6)
 			(drill 0.25)
-			(layers "F&B.Cu" "B.Mask")
+			(layers "*.Cu" "B.Mask")
 			(remove_unused_layers no)
 			(net 2 "GND")
@@
 			(size 0.6 0.6)
 			(drill 0.25)
-			(layers "F&B.Cu" "B.Mask")
+			(layers "*.Cu" "B.Mask")
 			(remove_unused_layers no)
 			(net 2 "GND")
@@
 			(size 0.6 0.6)
 			(drill 0.25)
-			(layers "F&B.Cu" "B.Mask")
+			(layers "*.Cu" "B.Mask")
 			(remove_unused_layers no)
 			(net 2 "GND")
@@
 			(size 0.6 0.6)
 			(drill 0.25)
-			(layers "F&B.Cu" "B.Mask")
+			(layers "*.Cu" "B.Mask")
 			(remove_unused_layers no)
 			(net 2 "GND")
@@
 			(size 0.6 0.6)
 			(drill 0.25)
-			(layers "F&B.Cu" "B.Mask")
+			(layers "*.Cu" "B.Mask")
 			(remove_unused_layers no)
 			(net 2 "GND")
@@
 			(size 0.6 0.6)
 			(drill 0.25)
-			(layers "F&B.Cu" "B.Mask")
+			(layers "*.Cu" "B.Mask")
 			(remove_unused_layers no)
 			(net 2 "GND")
@@
 			(size 0.6 0.6)
 			(drill 0.25)
-			(layers "F&B.Cu" "B.Mask")
+			(layers "*.Cu" "B.Mask")
 			(remove_unused_layers no)
 			(net 2 "GND")
@@
 			(size 0.6 0.6)
 			(drill 0.25)
-			(layers "F&B.Cu" "B.Mask")
+			(layers "*.Cu" "B.Mask")
 			(remove_unused_layers no)
 			(net 2 "GND")
@@
 			(size 0.6 0.6)
 			(drill 0.25)
-			(layers "F&B.Cu" "B.Mask")
+			(layers "*.Cu" "B.Mask")
 			(remove_unused_layers no)
 			(net 2 "GND")
@@
 			(size 2.775 2.775)
 			(drill 1.85)
-			(layers "F&B.Cu" "*.Mask")
+			(layers "*.Cu" "*.Mask")
 			(remove_unused_layers no)
 			(net 1 "+BATT")
@@
 			(size 2.775 2.775)
 			(drill 1.85)
-			(layers "F&B.Cu" "*.Mask")
+			(layers "*.Cu" "*.Mask")
 			(remove_unused_layers no)
 			(net 1 "+BATT")
@@
 			(drill oval 0.6 1.4)
 			(property pad_prop_heatsink)
-			(layers "F&B.Cu" "*.Mask")
+			(layers "*.Cu" "*.Mask")
 			(remove_unused_layers no)
 			(net 2 "GND")
@@
 			(drill oval 0.6 1.7)
 			(property pad_prop_heatsink)
-			(layers "F&B.Cu" "*.Mask")
+			(layers "*.Cu" "*.Mask")
 			(remove_unused_layers no)
 			(net 2 "GND")
@@
 			(drill oval 0.6 1.4)
 			(property pad_prop_heatsink)
-			(layers "F&B.Cu" "*.Mask")
+			(layers "*.Cu" "*.Mask")
 			(remove_unused_layers no)
 			(net 2 "GND")
@@
 			(drill oval 0.6 1.7)
 			(property pad_prop_heatsink)
-			(layers "F&B.Cu" "*.Mask")
+			(layers "*.Cu" "*.Mask")
 			(remove_unused_layers no)
 			(net 2 "GND")
@@
 			(size 1.24 1.24)
 			(drill 0.84)
-			(layers "F&B.Cu" "*.Mask")
+			(layers "*.Cu" "*.Mask")
 			(remove_unused_layers no)
 			(net 60 "/GPS/ANT")
@@
 			(size 1.24 1.24)
 			(drill 0.84)
-			(layers "F&B.Cu" "*.Mask")
+			(layers "*.Cu" "*.Mask")
 			(remove_unused_layers no)
 			(net 2 "GND")
@@
 			(size 1.24 1.24)
 			(drill 0.84)
-			(layers "F&B.Cu" "*.Mask")
+			(layers "*.Cu" "*.Mask")
 			(remove_unused_layers no)
 			(net 2 "GND")
@@
 			(size 1.24 1.24)
 			(drill 0.84)
-			(layers "F&B.Cu" "*.Mask")
+			(layers "*.Cu" "*.Mask")
 			(remove_unused_layers no)
 			(net 2 "GND")
@@
 			(size 1.24 1.24)
 			(drill 0.84)
-			(layers "F&B.Cu" "*.Mask")
+			(layers "*.Cu" "*.Mask")
 			(remove_unused_layers no)
 			(net 2 "GND")
@@
 		)
 	)
-	(gr_text "Ordering notes:\n4 layers, 1oz outer 1oz inner. Specify stackup so that In2.Cu is directly above B.Cu to ensure proper grounding of impedance controlled traces\nUse JLC 4 layer controlled stackup JLC041611-7628\nMin via size 0.25/0.4mm, order with vias epoxy filled and capped\nRemove Mark and please order it in something other than Green or Yellow"
+	(gr_text "Ordering notes:\nSpecify stackup so that In2.Cu is directly above B.Cu to ensure proper grounding of impedance controlled traces\nUse JLC 4 layer controlled stackup JLC04161H-7628 (default stackup)\nMin via size 0.25/0.4mm, order with vias epoxy filled and capped"
 		(at 13.4 71.8 0)
 		(layer "F.Fab")
@@
 	)
 	(segment
-		(start 128 36.25)
-		(end 131.75 36.25)
-		(width 0.286258)
+		(start 131.75 36.25)
+		(end 131.8 36.2)
+		(width 0.295402)
 		(layer "B.Cu")
 		(net 60)
 	)
 	(segment
-		(start 131.75 36.25)
-		(end 131.8 36.2)
-		(width 0.286258)
+		(start 128 36.25)
+		(end 131.75 36.25)
+		(width 0.295402)
 		(layer "B.Cu")
 		(net 60)
@@
 	)
 	(segment
-		(start 65.483379 44.798705)
-		(end 25.927695 44.798705)
-		(width 0.19939)
+		(start 67.713453 45.296546)
+		(end 65.984274 45.296546)
+		(width 0.203708)
 		(layer "B.Cu")
 		(net 85)
 	)
 	(segment
-		(start 24.634806 44.472305)
-		(end 24.625001 44.4625)
-		(width 0.19939)
+		(start 68.009999 45)
+		(end 67.713453 45.296546)
+		(width 0.203708)
 		(layer "B.Cu")
 		(net 85)
 	)
 	(segment
-		(start 24.625001 44.4625)
-		(end 24.25 44.4625)
-		(width 0.19939)
+		(start 25.929854 44.780527)
+		(end 25.619473 44.470146)
+		(width 0.203708)
 		(layer "B.Cu")
 		(net 85)
 	)
 	(segment
-		(start 25.618579 44.472305)
-		(end 24.634806 44.472305)
-		(width 0.19939)
+		(start 68.49 45)
+		(end 68.009999 45)
+		(width 0.203708)
 		(layer "B.Cu")
 		(net 85)
 	)
 	(segment
-		(start 68.49 45)
-		(end 68.196296 45.293704)
-		(width 0.19939)
+		(start 25.619473 44.470146)
+		(end 24.632647 44.470146)
+		(width 0.203708)
+		(layer "B.Cu")
+		(net 85)
+	)
+	(segment
+		(start 65.984274 45.296546)
+		(end 65.484274 44.796546)
+		(width 0.203708)
 		(layer "B.Cu")
 		(net 85)
 	)
 	(segment
-		(start 25.927695 44.798705)
-		(end 25.927695 44.781421)
-		(width 0.19939)
+		(start 25.929854 44.796546)
+		(end 25.929854 44.780527)
+		(width 0.203708)
 		(layer "B.Cu")
 		(net 85)
 	)
 	(segment
-		(start 65.978378 45.293704)
-		(end 65.483379 44.798705)
-		(width 0.19939)
+		(start 24.625001 44.4625)
+		(end 24.25 44.4625)
+		(width 0.203708)
 		(layer "B.Cu")
 		(net 85)
 	)
 	(segment
-		(start 25.927695 44.781421)
-		(end 25.618579 44.472305)
-		(width 0.19939)
+		(start 65.484274 44.796546)
+		(end 25.929854 44.796546)
+		(width 0.203708)
 		(layer "B.Cu")
 		(net 85)
 	)
 	(segment
-		(start 68.196296 45.293704)
-		(end 65.978378 45.293704)
-		(width 0.19939)
+		(start 24.632647 44.470146)
+		(end 24.625001 44.4625)
+		(width 0.203708)
 		(layer "B.Cu")
 		(net 85)
 	)
 	(segment
-		(start 65.811622 45.696296)
-		(end 65.316621 45.201295)
-		(width 0.19939)
+		(start 65.815726 45.703454)
+		(end 65.315726 45.203454)
+		(width 0.203708)
 		(layer "B.Cu")
 		(net 86)
 	)
 	(segment
-		(start 24.625001 45.5375)
-		(end 24.25 45.5375)
-		(width 0.19939)
+		(start 67.713453 45.703454)
+		(end 65.815726 45.703454)
+		(width 0.203708)
 		(layer "B.Cu")
 		(net 86)
 	)
 	(segment
-		(start 25.927695 45.201295)
-		(end 25.927695 45.218579)
-		(width 0.19939)
+		(start 65.315726 45.203454)
+		(end 25.929854 45.203454)
+		(width 0.203708)
 		(layer "B.Cu")
 		(net 86)
 	)
 	(segment
-		(start 68.196296 45.696296)
-		(end 65.811622 45.696296)
-		(width 0.19939)
+		(start 25.929854 45.203454)
+		(end 25.929854 45.219473)
+		(width 0.203708)
 		(layer "B.Cu")
 		(net 86)
 	)
 	(segment
-		(start 25.927695 45.218579)
-		(end 25.618579 45.527695)
-		(width 0.19939)
+		(start 25.929854 45.219473)
+		(end 25.619473 45.529854)
+		(width 0.203708)
 		(layer "B.Cu")
 		(net 86)
 	)
 	(segment
-		(start 24.634806 45.527695)
-		(end 24.625001 45.5375)
-		(width 0.19939)
+		(start 25.619473 45.529854)
+		(end 24.632647 45.529854)
+		(width 0.203708)
 		(layer "B.Cu")
 		(net 86)
 	)
 	(segment
-		(start 68.5 46)
-		(end 68.196296 45.696296)
-		(width 0.19939)
+		(start 68.49 46)
+		(end 68.009999 46)
+		(width 0.203708)
 		(layer "B.Cu")
 		(net 86)
 	)
 	(segment
-		(start 25.618579 45.527695)
-		(end 24.634806 45.527695)
-		(width 0.19939)
+		(start 68.009999 46)
+		(end 67.713453 45.703454)
+		(width 0.203708)
 		(layer "B.Cu")
 		(net 86)
 	)
 	(segment
-		(start 65.316621 45.201295)
-		(end 25.927695 45.201295)
-		(width 0.19939)
+		(start 24.632647 45.529854)
+		(end 24.625001 45.5375)
+		(width 0.203708)
 		(layer "B.Cu")
 		(net 86)
 	)
 	(segment
-		(start 70.1545 46.6345)
-		(end 69.52 46)
-		(width 0.2)
+		(start 24.625001 45.5375)
+		(end 24.25 45.5375)
+		(width 0.203708)
 		(layer "B.Cu")
-		(net 87)
+		(net 86)
 	)
 	(segment
@@
 		(width 0.2)
 		(layer "B.Cu")
+		(net 87)
+	)
+	(segment
+		(start 69.52 46)
+		(end 69.51 46)
+		(width 0.2)
+		(layer "B.Cu")
+		(net 87)
+	)
+	(segment
+		(start 70.1545 46.6345)
+		(end 69.52 46)
+		(width 0.2)
+		(layer "B.Cu")
