File: precision-clock-pcb/rtc.kicad_sch (KiCad schematic)
At the start: 1 part, among them U4 DS3232M

Commit message: schematic work done
Parts:
- added BT1: CR2012, symbol Device:Battery_Cell
- added C25: 100nF, symbol Device:C
- added C26, C28: 1uF, symbol Device:C
- added Q13: BSS83P, Package_TO_SOT_SMD:SOT-23, symbol Transistor_FET:BSS83P
- added Q14: BSS138, Package_TO_SOT_SMD:SOT-23, symbol Transistor_FET:BSS138
- added R39, R44: 100K, symbol Device:R
- added R40, R41: 4.7K, symbol Device:R
- added R43: 1M, symbol Device:R
- added TP1: TestPoint, symbol Connector:TestPoint
Connections:
- net at U4.1 (32KHZ): now also TP1.1
- net +3V3: now reaches U4.2 (VCC)
- net +3V3: now also C25.1, C26.1, R39.2, R40.2, R41.2
- net at U4.3 (~{INT}/SQW): now also R39.1
- net RST: now reaches U4.4 (~{RST})
- net GND: now reaches U4.5 (GND)
- net GND: now also BT1.2 (-), C25.2, C26.2, C28.2, Q14.2 (S), R44.1
- net +BATT: now reaches U4.6 (VBAT)
- net +BATT: now also BT1.1 (+), Q13.3 (D), R43.1
- net SDA: now reaches U4.7 (SDA)
- net SDA: now also R41.1
- net SCL: now reaches U4.8 (SCL)
- net SCL: now also R40.1
- new net: Q13.1 (G), Q14.3 (D), R43.2
- new net BATT_SENSE: C28.1, Q13.2 (S)
- new net BAT_GATE_EN: Q14.1 (G), R44.2

Commit message: board work
Parts:
- BT1: value CR2012 -> CR1220; footprint (none) -> Battery_Custom:BAT_2895
- C27: renamed from C28; footprint (none) -> Capacitor_SMD:C_0603_1608Metric
- C28: renamed from C25; footprint (none) -> Capacitor_SMD:C_0402_1005Metric
- C29: renamed from C26; footprint (none) -> Capacitor_SMD:C_0603_1608Metric
- R22: renamed from R44; footprint (none) -> Resistor_SMD:R_0402_1005Metric
- R23: renamed from R43; footprint (none) -> Resistor_SMD:R_0402_1005Metric
- R24: renamed from R41; footprint (none) -> Resistor_SMD:R_0402_1005Metric
- R25: renamed from R40; footprint (none) -> Resistor_SMD:R_0402_1005Metric
- R26: renamed from R39; footprint (none) -> Resistor_SMD:R_0402_1005Metric
- TP1: footprint (none) -> TestPoint:TestPoint_Pad_2.0x2.0mm
- renumbered Q14 to Q3, Q13 to Q4, U4 to U6
Changed lines of the file:
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@@
 		(on_board yes)
 		(dnp no)
-		(property "Reference" "#PWR046"
+		(property "Reference" "#PWR043"
 			(at 77.47 68.58 0)
 			(effects
@@
 			(project "precision-clock"
 				(path "/3cbd0e8e-3ba4-43b1-82ac-749e7a469b5f/b1d4eb23-a2bb-480a-90a1-dafbdf84a746"
-					(reference "#PWR046")
+					(reference "#PWR043")
 					(unit 1)
 				)
@@
 		(dnp no)
 		(fields_autoplaced yes)
-		(property "Reference" "Q14"
+		(property "Reference" "Q3"
 			(at 93.98 66.0399 0)
 			(effects
@@
 			(project ""
 				(path "/3cbd0e8e-3ba4-43b1-82ac-749e7a469b5f/b1d4eb23-a2bb-480a-90a1-dafbdf84a746"
-					(reference "Q14")
+					(reference "Q3")
 					(unit 1)
 				)
@@
 		(dnp no)
 		(fields_autoplaced yes)
-		(property "Reference" "C26"
+		(property "Reference" "C29"
 			(at 151.13 62.2299 0)
 			(effects
@@
 			)
 		)
-		(property "Footprint" ""
+		(property "Footprint" "Capacitor_SMD:C_0603_1608Metric"
 			(at 148.2852 67.31 0)
 			(effects
@@
 			(project "precision-clock"
 				(path "/3cbd0e8e-3ba4-43b1-82ac-749e7a469b5f/b1d4eb23-a2bb-480a-90a1-dafbdf84a746"
-					(reference "C26")
+					(reference "C29")
 					(unit 1)
 				)
@@
 		(on_board yes)
 		(dnp no)
-		(property "Reference" "R41"
+		(property "Reference" "R24"
 			(at 104.394 78.74 0)
 			(effects
@@
 			)
 		)
-		(property "Footprint" ""
+		(property "Footprint" "Resistor_SMD:R_0402_1005Metric"
 			(at 104.648 78.74 90)
 			(effects
@@
 			(project "precision-clock"
 				(path "/3cbd0e8e-3ba4-43b1-82ac-749e7a469b5f/b1d4eb23-a2bb-480a-90a1-dafbdf84a746"
-					(reference "R41")
+					(reference "R24")
 					(unit 1)
 				)
@@
 		(dnp no)
 		(fields_autoplaced yes)
-		(property "Reference" "C28"
+		(property "Reference" "C27"
 			(at 81.28 57.1499 0)
 			(effects
@@
 			)
 		)
-		(property "Footprint" ""
+		(property "Footprint" "Capacitor_SMD:C_0603_1608Metric"
 			(at 78.4352 62.23 0)
 			(effects
@@
 			(project "precision-clock"
 				(path "/3cbd0e8e-3ba4-43b1-82ac-749e7a469b5f/b1d4eb23-a2bb-480a-90a1-dafbdf84a746"
-					(reference "C28")
+					(reference "C27")
 					(unit 1)
 				)
@@
 		(dnp no)
 		(fields_autoplaced yes)
-		(property "Reference" "U4"
+		(property "Reference" "U6"
 			(at 131.6833 96.52 0)
 			(effects
@@
 			(project "precision-clock"
 				(path "/3cbd0e8e-3ba4-43b1-82ac-749e7a469b5f/b1d4eb23-a2bb-480a-90a1-dafbdf84a746"
-					(reference "U4")
+					(reference "U6")
 					(unit 1)
 				)
@@
 		(on_board yes)
 		(dnp no)
-		(property "Reference" "R39"
+		(property "Reference" "R26"
 			(at 146.05 86.614 90)
 			(effects
@@
 			)
 		)
-		(property "Footprint" ""
+		(property "Footprint" "Resistor_SMD:R_0402_1005Metric"
 			(at 146.05 90.678 90)
 			(effects
@@
 			(project ""
 				(path "/3cbd0e8e-3ba4-43b1-82ac-749e7a469b5f/b1d4eb23-a2bb-480a-90a1-dafbdf84a746"
-					(reference "R39")
+					(reference "R26")
 					(unit 1)
 				)
@@
 			)
 		)
-		(property "Value" "CR2012"
+		(property "Value" "CR1220"
 			(at 110.49 59.1184 0)
 			(effects
@@
 			)
 		)
-		(property "Footprint" ""
+		(property "Footprint" "Battery_Custom:BAT_2895"
 			(at 106.68 58.166 90)
 			(effects
@@
 		(on_board yes)
 		(dnp no)
-		(property "Reference" "#PWR038"
+		(property "Reference" "#PWR046"
 			(at 102.87 77.47 0)
 			(effects
@@
 			(project "precision-clock"
 				(path "/3cbd0e8e-3ba4-43b1-82ac-749e7a469b5f/b1d4eb23-a2bb-480a-90a1-dafbdf84a746"
-					(reference "#PWR038")
+					(reference "#PWR046")
 					(unit 1)
 				)
@@
 		(dnp no)
 		(fields_autoplaced yes)
-		(property "Reference" "Q13"
+		(property "Reference" "Q4"
 			(at 90.17 48.26 90)
 			(effects
@@
 			(project ""
 				(path "/3cbd0e8e-3ba4-43b1-82ac-749e7a469b5f/b1d4eb23-a2bb-480a-90a1-dafbdf84a746"
-					(reference "Q13")
+					(reference "Q4")
 					(unit 1)
 				)
@@
 			)
 		)
-		(property "Footprint" ""
+		(property "Footprint" "TestPoint:TestPoint_Pad_2.0x2.0mm"
 			(at 157.48 81.28 0)
 			(effects
@@
 		(on_board yes)
 		(dnp no)
-		(property "Reference" "#PWR037"
+		(property "Reference" "#PWR052"
 			(at 152.4 92.71 0)
 			(effects
@@
 			(project "precision-clock"
 				(path "/3cbd0e8e-3ba4-43b1-82ac-749e7a469b5f/b1d4eb23-a2bb-480a-90a1-dafbdf84a746"
-					(reference "#PWR037")
+					(reference "#PWR052")
 					(unit 1)
 				)
@@
 		(dnp no)
 		(fields_autoplaced yes)
-		(property "Reference" "#PWR033"
+		(property "Reference" "#PWR049"
 			(at 129.54 102.87 0)
 			(effects
@@
 			(project ""
 				(path "/3cbd0e8e-3ba4-43b1-82ac-749e7a469b5f/b1d4eb23-a2bb-480a-90a1-dafbdf84a746"
-					(reference "#PWR033")
+					(reference "#PWR049")
 					(unit 1)
 				)
@@
 		(dnp no)
 		(fields_autoplaced yes)
-		(property "Reference" "#PWR036"
+		(property "Reference" "#PWR051"
 			(at 147.32 73.66 0)
 			(effects
@@
 			(project "precision-clock"
 				(path "/3cbd0e8e-3ba4-43b1-82ac-749e7a469b5f/b1d4eb23-a2bb-480a-90a1-dafbdf84a746"
-					(reference "#PWR036")
+					(reference "#PWR051")
 					(unit 1)
 				)
@@
 		(on_board yes)
 		(dnp no)
-		(property "Reference" "R40"
+		(property "Reference" "R25"
 			(at 112.014 77.47 0)
 			(effects
@@
 			)
 		)
-		(property "Footprint" ""
+		(property "Footprint" "Resistor_SMD:R_0402_1005Metric"
 			(at 112.268 77.47 90)
 			(effects
@@
 			(project "precision-clock"
 				(path "/3cbd0e8e-3ba4-43b1-82ac-749e7a469b5f/b1d4eb23-a2bb-480a-90a1-dafbdf84a746"
-					(reference "R40")
+					(reference "R25")
 					(unit 1)
 				)
@@
 		(on_board yes)
 		(dnp no)
-		(property "Reference" "#PWR032"
+		(property "Reference" "#PWR050"
 			(at 147.32 63.5 0)
 			(effects
@@
 			(project "precision-clock"
 				(path "/3cbd0e8e-3ba4-43b1-82ac-749e7a469b5f/b1d4eb23-a2bb-480a-90a1-dafbdf84a746"
-					(reference "#PWR032")
+					(reference "#PWR050")
 					(unit 1)
 				)
@@
 		(dnp no)
 		(fields_autoplaced yes)
-		(property "Reference" "#PWR035"
+		(property "Reference" "#PWR048"
 			(at 106.68 68.58 0)
 			(effects
@@
 			(project "precision-clock"
 				(path "/3cbd0e8e-3ba4-43b1-82ac-749e7a469b5f/b1d4eb23-a2bb-480a-90a1-dafbdf84a746"
-					(reference "#PWR035")
+					(reference "#PWR048")
 					(unit 1)
 				)
@@
 		(dnp no)
 		(fields_autoplaced yes)
-		(property "Reference" "#PWR045"
+		(property "Reference" "#PWR044"
 			(at 82.55 81.28 0)
 			(effects
@@
 			(project "precision-clock"
 				(path "/3cbd0e8e-3ba4-43b1-82ac-749e7a469b5f/b1d4eb23-a2bb-480a-90a1-dafbdf84a746"
-					(reference "#PWR045")
+					(reference "#PWR044")
 					(unit 1)
 				)
@@
 		(dnp no)
 		(fields_autoplaced yes)
-		(property "Reference" "#PWR044"
+		(property "Reference" "#PWR045"
 			(at 90.17 78.74 0)
 			(effects
@@
 			(project "precision-clock"
 				(path "/3cbd0e8e-3ba4-43b1-82ac-749e7a469b5f/b1d4eb23-a2bb-480a-90a1-dafbdf84a746"
-					(reference "#PWR044")
+					(reference "#PWR045")
 					(unit 1)
 				)
@@
 		(on_board yes)
 		(dnp no)
-		(property "Reference" "R44"
+		(property "Reference" "R22"
 			(at 79.502 71.12 0)
 			(effects
@@
 			)
 		)
-		(property "Footprint" ""
+		(property "Footprint" "Resistor_SMD:R_0402_1005Metric"
 			(at 84.328 71.12 90)
 			(effects
@@
 			(project "precision-clock"
 				(path "/3cbd0e8e-3ba4-43b1-82ac-749e7a469b5f/b1d4eb23-a2bb-480a-90a1-dafbdf84a746"
-					(reference "R44")
+					(reference "R22")
 					(unit 1)
 				)
@@
 		(dnp no)
 		(fields_autoplaced yes)
-		(property "Reference" "#PWR034"
+		(property "Reference" "#PWR047"
 			(at 106.68 58.42 0)
 			(effects
@@
 			(project ""
 				(path "/3cbd0e8e-3ba4-43b1-82ac-749e7a469b5f/b1d4eb23-a2bb-480a-90a1-dafbdf84a746"
-					(reference "#PWR034")
+					(reference "#PWR047")
 					(unit 1)
 				)
@@
 		(dnp no)
 		(fields_autoplaced yes)
-		(property "Reference" "C25"
+		(property "Reference" "C28"
 			(at 137.16 62.2299 0)
 			(effects
@@
 			)
 		)
-		(property "Footprint" ""
+		(property "Footprint" "Capacitor_SMD:C_0402_1005Metric"
 			(at 134.3152 67.31 0)
 			(effects
@@
 			(project ""
 				(path "/3cbd0e8e-3ba4-43b1-82ac-749e7a469b5f/b1d4eb23-a2bb-480a-90a1-dafbdf84a746"
-					(reference "C25")
+					(reference "C28")
 					(unit 1)
 				)
@@
 		(on_board yes)
 		(dnp no)
-		(property "Reference" "R43"
+		(property "Reference" "R23"
 			(at 97.536 58.42 90)
 			(effects
@@
 			)
 		)
-		(property "Footprint" ""
+		(property "Footprint" "Resistor_SMD:R_0402_1005Metric"
 			(at 93.472 58.42 90)
 			(effects
@@
 			(project "precision-clock"
 				(path "/3cbd0e8e-3ba4-43b1-82ac-749e7a469b5f/b1d4eb23-a2bb-480a-90a1-dafbdf84a746"
-					(reference "R43")
-					(unit 1)
-				)
+					(reference "R23")
+					(unit 1)
+				)

Commit message: board work
Parts:
- renumbered Q4 to Q3, Q3 to Q4, R23 to R22, R22 to R23, R25 to R24, R24 to R25
Changed lines of the file:
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@@
 		(on_board yes)
 		(dnp no)
-		(property "Reference" "#PWR043"
+		(property "Reference" "#PWR045"
 			(at 77.47 68.58 0)
 			(effects
@@
 			(project "precision-clock"
 				(path "/3cbd0e8e-3ba4-43b1-82ac-749e7a469b5f/b1d4eb23-a2bb-480a-90a1-dafbdf84a746"
-					(reference "#PWR043")
+					(reference "#PWR045")
 					(unit 1)
 				)
@@
 		(dnp no)
 		(fields_autoplaced yes)
-		(property "Reference" "Q3"
+		(property "Reference" "Q4"
 			(at 93.98 66.0399 0)
 			(effects
@@
 			(project ""
 				(path "/3cbd0e8e-3ba4-43b1-82ac-749e7a469b5f/b1d4eb23-a2bb-480a-90a1-dafbdf84a746"
-					(reference "Q3")
+					(reference "Q4")
 					(unit 1)
 				)
@@
 		(on_board yes)
 		(dnp no)
-		(property "Reference" "R24"
+		(property "Reference" "R25"
 			(at 104.394 78.74 0)
 			(effects
@@
 			(project "precision-clock"
 				(path "/3cbd0e8e-3ba4-43b1-82ac-749e7a469b5f/b1d4eb23-a2bb-480a-90a1-dafbdf84a746"
-					(reference "R24")
+					(reference "R25")
 					(unit 1)
 				)
@@
 		(on_board yes)
 		(dnp no)
-		(property "Reference" "#PWR046"
+		(property "Reference" "#PWR049"
 			(at 102.87 77.47 0)
 			(effects
@@
 			(project "precision-clock"
 				(path "/3cbd0e8e-3ba4-43b1-82ac-749e7a469b5f/b1d4eb23-a2bb-480a-90a1-dafbdf84a746"
-					(reference "#PWR046")
+					(reference "#PWR049")
 					(unit 1)
 				)
@@
 		(dnp no)
 		(fields_autoplaced yes)
-		(property "Reference" "Q4"
+		(property "Reference" "Q3"
 			(at 90.17 48.26 90)
 			(effects
@@
 			(project ""
 				(path "/3cbd0e8e-3ba4-43b1-82ac-749e7a469b5f/b1d4eb23-a2bb-480a-90a1-dafbdf84a746"
-					(reference "Q4")
+					(reference "Q3")
 					(unit 1)
 				)
@@
 		(on_board yes)
 		(dnp no)
-		(property "Reference" "#PWR052"
+		(property "Reference" "#PWR051"
 			(at 152.4 92.71 0)
 			(effects
@@
 			(project "precision-clock"
 				(path "/3cbd0e8e-3ba4-43b1-82ac-749e7a469b5f/b1d4eb23-a2bb-480a-90a1-dafbdf84a746"
-					(reference "#PWR052")
+					(reference "#PWR051")
 					(unit 1)
 				)
@@
 		(dnp no)
 		(fields_autoplaced yes)
-		(property "Reference" "#PWR049"
+		(property "Reference" "#PWR052"
 			(at 129.54 102.87 0)
 			(effects
@@
 			(project ""
 				(path "/3cbd0e8e-3ba4-43b1-82ac-749e7a469b5f/b1d4eb23-a2bb-480a-90a1-dafbdf84a746"
-					(reference "#PWR049")
+					(reference "#PWR052")
 					(unit 1)
 				)
@@
 		(dnp no)
 		(fields_autoplaced yes)
-		(property "Reference" "#PWR051"
+		(property "Reference" "#PWR047"
 			(at 147.32 73.66 0)
 			(effects
@@
 			(project "precision-clock"
 				(path "/3cbd0e8e-3ba4-43b1-82ac-749e7a469b5f/b1d4eb23-a2bb-480a-90a1-dafbdf84a746"
-					(reference "#PWR051")
+					(reference "#PWR047")
 					(unit 1)
 				)
@@
 		(on_board yes)
 		(dnp no)
-		(property "Reference" "R25"
+		(property "Reference" "R24"
 			(at 112.014 77.47 0)
 			(effects
@@
 			(project "precision-clock"
 				(path "/3cbd0e8e-3ba4-43b1-82ac-749e7a469b5f/b1d4eb23-a2bb-480a-90a1-dafbdf84a746"
-					(reference "R25")
+					(reference "R24")
 					(unit 1)
 				)
@@
 		(on_board yes)
 		(dnp no)
-		(property "Reference" "#PWR050"
+		(property "Reference" "#PWR044"
 			(at 147.32 63.5 0)
 			(effects
@@
 			(project "precision-clock"
 				(path "/3cbd0e8e-3ba4-43b1-82ac-749e7a469b5f/b1d4eb23-a2bb-480a-90a1-dafbdf84a746"
-					(reference "#PWR050")
+					(reference "#PWR044")
 					(unit 1)
 				)
@@
 		(dnp no)
 		(fields_autoplaced yes)
-		(property "Reference" "#PWR048"
+		(property "Reference" "#PWR046"
 			(at 106.68 68.58 0)
 			(effects
@@
 			(project "precision-clock"
 				(path "/3cbd0e8e-3ba4-43b1-82ac-749e7a469b5f/b1d4eb23-a2bb-480a-90a1-dafbdf84a746"
-					(reference "#PWR048")
+					(reference "#PWR046")
 					(unit 1)
 				)
@@
 		(dnp no)
 		(fields_autoplaced yes)
-		(property "Reference" "#PWR044"
+		(property "Reference" "#PWR050"
 			(at 82.55 81.28 0)
 			(effects
@@
 			(project "precision-clock"
 				(path "/3cbd0e8e-3ba4-43b1-82ac-749e7a469b5f/b1d4eb23-a2bb-480a-90a1-dafbdf84a746"
-					(reference "#PWR044")
+					(reference "#PWR050")
 					(unit 1)
 				)
@@
 		(dnp no)
 		(fields_autoplaced yes)
-		(property "Reference" "#PWR045"
+		(property "Reference" "#PWR048"
 			(at 90.17 78.74 0)
 			(effects
@@
 			(project "precision-clock"
 				(path "/3cbd0e8e-3ba4-43b1-82ac-749e7a469b5f/b1d4eb23-a2bb-480a-90a1-dafbdf84a746"
-					(reference "#PWR045")
+					(reference "#PWR048")
 					(unit 1)
 				)
@@
 		(on_board yes)
 		(dnp no)
-		(property "Reference" "R22"
+		(property "Reference" "R23"
 			(at 79.502 71.12 0)
 			(effects
@@
 			(project "precision-clock"
 				(path "/3cbd0e8e-3ba4-43b1-82ac-749e7a469b5f/b1d4eb23-a2bb-480a-90a1-dafbdf84a746"
-					(reference "R22")
+					(reference "R23")
 					(unit 1)
 				)
@@
 		(dnp no)
 		(fields_autoplaced yes)
-		(property "Reference" "#PWR047"
+		(property "Reference" "#PWR043"
 			(at 106.68 58.42 0)
 			(effects
@@
 			(project ""
 				(path "/3cbd0e8e-3ba4-43b1-82ac-749e7a469b5f/b1d4eb23-a2bb-480a-90a1-dafbdf84a746"
-					(reference "#PWR047")
+					(reference "#PWR043")
 					(unit 1)
 				)
@@
 		(on_board yes)
 		(dnp no)
-		(property "Reference" "R23"
+		(property "Reference" "R22"
 			(at 97.536 58.42 90)
 			(effects
@@
 			(project "precision-clock"
 				(path "/3cbd0e8e-3ba4-43b1-82ac-749e7a469b5f/b1d4eb23-a2bb-480a-90a1-dafbdf84a746"
-					(reference "R23")
-					(unit 1)
-				)
+					(reference "R22")
+					(unit 1)
+				)

Commit message: BOM, CSV, and STEP exports
Parts:
- BT1: JLCPCB PN (none) -> C5495443; MFR PN (none) -> 2895
- C27, C29: JLCPCB PN (none) -> C29936; MFR PN (none) -> CL10B105KA8NNNC
- C28: JLCPCB PN (none) -> C77014; MFR PN (none) -> GRM155R71E104KE14D
- Q3: JLCPCB PN (none) -> C2932927; MFR PN (none) -> BSS83PH6327
- Q4: JLCPCB PN (none) -> C52895; MFR PN (none) -> BSS138
- R22: JLCPCB PN (none) -> C138033; MFR PN (none) -> RC0402FR-071ML
- R23, R26: JLCPCB PN (none) -> C60491; MFR PN (none) -> RC0402FR-07100KL
- R24, R25: JLCPCB PN (none) -> C105871; MFR PN (none) -> RC0402FR-074K7L
- U6: JLCPCB PN (none) -> C2827535; MFR PN (none) -> DS3232MZ+TRL
Changed lines of the file:
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@@
+			)
+		)
+		(property "JLCPCB PN" "C52895"
+			(at 87.63 67.31 0)
+			(effects
+				(font
+					(size 1.27 1.27)
+				)
+				(hide yes)
+			)
+		)
+		(property "MFR PN" "BSS138"
+			(at 87.63 67.31 0)
+			(effects
+				(font
+					(size 1.27 1.27)
+				)
+				(hide yes)
 			)
 		)
@@
 			)
 		)
+		(property "JLCPCB PN" "C29936 "
+			(at 147.32 63.5 0)
+			(effects
+				(font
+					(size 1.27 1.27)
+				)
+				(hide yes)
+			)
+		)
+		(property "MFR PN" "CL10B105KA8NNNC"
+			(at 147.32 63.5 0)
+			(effects
+				(font
+					(size 1.27 1.27)
+				)
+				(hide yes)
+			)
+		)
 		(pin "1"
 		)
@@
 		)
 		(property "Description" "Resistor"
+			(at 102.87 78.74 0)
+			(effects
+				(font
+					(size 1.27 1.27)
+				)
+				(hide yes)
+			)
+		)
+		(property "JLCPCB PN" "C105871"
+			(at 102.87 78.74 0)
+			(effects
+				(font
+					(size 1.27 1.27)
+				)
+				(hide yes)
+			)
+		)
+		(property "MFR PN" "RC0402FR-074K7L"
 			(at 102.87 78.74 0)
 			(effects
@@
 			)
 		)
+		(property "JLCPCB PN" "C29936 "
+			(at 77.47 58.42 0)
+			(effects
+				(font
+					(size 1.27 1.27)
+				)
+				(hide yes)
+			)
+		)
+		(property "MFR PN" "CL10B105KA8NNNC"
+			(at 77.47 58.42 0)
+			(effects
+				(font
+					(size 1.27 1.27)
+				)
+				(hide yes)
+			)
+		)
 		(pin "1"
 		)
@@
 			)
 		)
+		(property "JLCPCB PN" "C2827535"
+			(at 129.54 86.36 0)
+			(effects
+				(font
+					(size 1.27 1.27)
+				)
+				(hide yes)
+			)
+		)
+		(property "MFR PN" "DS3232MZ+TRL"
+			(at 129.54 86.36 0)
+			(effects
+				(font
+					(size 1.27 1.27)
+				)
+				(hide yes)
+			)
+		)
 		(pin "3"
 		)
@@
 		(property "Description" "Resistor"
 			(at 146.05 88.9 0)
+			(effects
+				(font
+					(size 1.27 1.27)
+				)
+				(hide yes)
+			)
+		)
+		(property "JLCPCB PN" "C60491 "
+			(at 146.05 88.9 90)
+			(effects
+				(font
+					(size 1.27 1.27)
+				)
+				(hide yes)
+			)
+		)
+		(property "MFR PN" "RC0402FR-07100KL"
+			(at 146.05 88.9 90)
 			(effects
 				(font
@@
 			)
 		)
+		(property "JLCPCB PN" "C5495443"
+			(at 106.68 59.69 0)
+			(effects
+				(font
+					(size 1.27 1.27)
+				)
+				(hide yes)
+			)
+		)
+		(property "MFR PN" "2895"
+			(at 106.68 59.69 0)
+			(effects
+				(font
+					(size 1.27 1.27)
+				)
+				(hide yes)
+			)
+		)
 		(pin "2"
 		)
@@
 			)
 		)
+		(property "JLCPCB PN" "C2932927"
+			(at 90.17 57.15 90)
+			(effects
+				(font
+					(size 1.27 1.27)
+				)
+				(hide yes)
+			)
+		)
+		(property "MFR PN" "BSS83PH6327"
+			(at 90.17 57.15 90)
+			(effects
+				(font
+					(size 1.27 1.27)
+				)
+				(hide yes)
+			)
+		)
 		(pin "2"
 		)
@@
 			)
 		)
+		(property "JLCPCB PN" ""
+			(at 152.4 81.28 0)
+			(effects
+				(font
+					(size 1.27 1.27)
+				)
+				(hide yes)
+			)
+		)
+		(property "MFR PN" ""
+			(at 152.4 81.28 0)
+			(effects
+				(font
+					(size 1.27 1.27)
+				)
+				(hide yes)
+			)
+		)
 		(pin "1"
 		)
@@
 			)
 		)
+		(property "JLCPCB PN" "C105871"
+			(at 110.49 77.47 0)
+			(effects
+				(font
+					(size 1.27 1.27)
+				)
+				(hide yes)
+			)
+		)
+		(property "MFR PN" "RC0402FR-074K7L"
+			(at 110.49 77.47 0)
+			(effects
+				(font
+					(size 1.27 1.27)
+				)
+				(hide yes)
+			)
+		)
 		(pin "1"
 		)
@@
 			)
 		)
+		(property "JLCPCB PN" "C60491 "
+			(at 82.55 71.12 0)
+			(effects
+				(font
+					(size 1.27 1.27)
+				)
+				(hide yes)
+			)
+		)
+		(property "MFR PN" "RC0402FR-07100KL"
+			(at 82.55 71.12 0)
+			(effects
+				(font
+					(size 1.27 1.27)
+				)
+				(hide yes)
+			)
+		)
 		(pin "1"
 		)
@@
 			)
 		)
+		(property "JLCPCB PN" "C77014"
+			(at 133.35 63.5 0)
+			(effects
+				(font
+					(size 1.27 1.27)
+				)
+				(hide yes)
+			)
+		)
+		(property "MFR PN" "GRM155R71E104KE14D"
+			(at 133.35 63.5 0)
+			(effects
+				(font
+					(size 1.27 1.27)
+				)
+				(hide yes)
+			)
+		)
 		(pin "1"
 		)
@@
 			(effects
 				(font
+					(size 1.27 1.27)
+				)
+				(hide yes)
+			)
+		)
+		(property "JLCPCB PN" "C138033 "
+			(at 95.25 58.42 90)
+			(effects
+				(font
+					(size 1.27 1.27)
+				)
+				(hide yes)
+			)
+		)
+		(property "MFR PN" "RC0402FR-071ML"
+			(at 95.25 58.42 90)
+			(effects
+				(font
