File: precision-clock-pcb/precision-clock.kicad_sch (KiCad schematic)
At the start: 38 parts, among them J1 USB_C_Receptacle_USB2.0_14P, SW1 BOOTSEL, SW2 RESET, U1 RP2350_80QFN, U2 W25Q128JVS, U3 NCP1117-3.3_SOT223, U9 USBLC6-2P6, Y1 ABM8-272-T3

Commit message: schematic work done
Parts:
- added C29, C30, C31, C32: 100nF, Capacitor_SMD:C_0402_1005Metric, symbol Device:C
- added J3: TC2050, Connector:Tag-Connect_TC2050-IDC-FP_2x05_P1.27mm_Vertical, symbol Connector:TC2050
- added Q15, Q16: SFH320, LED_SMD:LED_PLCC-2_3.4x3.0mm_KA, symbol Sensor_Optical:SFH320
- added R45, R46: 10K, symbol Device:R
- added R47, R48, R50, R51, R52: 1K, Resistor_SMD:R_0402_1005Metric, symbol Device:R
- added R49: 0R, Resistor_SMD:R_0402_1005Metric, symbol Device:R
- added SW3, SW4: BUTTON, Button_Switch_SMD:SW_SPST_PTS647_Sx38, symbol Switch:SW_Push
- C4, C7: value 10u -> 10uF
Connections:
- net +3V3: now also J3.4, Q15.1 (C), Q16.1 (C)
- net GND: now also SW2.1, C29.2, C30.2, C31.2, C32.2, J3.3, R45.2, R46.2, SW3.1, SW4.1; no longer R4.2
- net RUN: now also R4.1, R52.2; no longer SW2.2
- net SWCLK: now also R50.1
- net SWD: now also R51.1
- net UART0_RX: now also R47.1
- net UART0_TX: now also R48.1
- net DISPBUS05: now reaches U1.11 (GPIO12)
- net DISPBUS06: now reaches U1.12 (GPIO13)
- net DISPBUS07: now reaches U1.13 (GPIO14)
- net DISPBUS08: now reaches U1.14 (GPIO15)
- net DISPBUS09: now reaches U1.16 (GPIO16)
- net DISPBUS10: now reaches U1.17 (GPIO17)
- net DISPBUS11: now reaches U1.18 (GPIO18)
- net DISPBUS12: now reaches U1.19 (GPIO19)
- net DISPBUS13: now reaches U1.20 (GPIO20)
- net DISPBUS14: now reaches U1.21 (GPIO21)
- net DISPBUS15: now reaches U1.22 (GPIO22)
- net DISPBUS16: now reaches U1.23 (GPIO23)
- net DISPBUS17: now reaches U1.25 (GPIO24)
- net DISPBUS18: now reaches U1.26 (GPIO25)
- net DISPBUS19: now reaches U1.27 (GPIO26)
- net DISPBUS20: now reaches U1.28 (GPIO27)
- net DIGPWM: now reaches U1.36 (GPIO28)
- net DOTPWM: now reaches U1.37 (GPIO29)
- net BATT_READ_EN: now reaches U1.38 (GPIO30)
- net USER_BUTTON_1: now reaches U1.39 (GPIO31)
- net USER_BUTTON_1: now also C31.1, SW3.2
- net USER_BUTTON_2: now reaches U1.40 (GPIO32)
- net USER_BUTTON_2: now also C32.1, SW4.2
- net ADC0: now reaches U1.49 (GPIO40_ADC0)
- net PD1: now reaches U1.52 (GPIO41_ADC1)
- net PD1: now also C29.1, Q15.2 (E), R45.1
- net PD2: now reaches U1.53 (GPIO42_ADC2)
- net PD2: now also C30.1, Q16.2 (E), R46.1
- net DISPBUS01: now reaches U1.6 (GPIO8)
- net DISPBUS02: now reaches U1.7 (GPIO9)
- net PPS_IN: now reaches U1.79 (GPIO2)
- net DISPBUS03: now reaches U1.8 (GPIO10)
- net DISPBUS04: now reaches U1.9 (GPIO11)
- net VBUS renamed +5V
- net +5V: now also R49.2
- new net: J3.5, R49.1
- new net: R4.2, SW2.2
- new net: J3.1, R52.1
- new net: J3.10, R50.2
- new net: J3.7, R48.2
- new net: J3.8, R47.2
- new net: J3.9, R51.2
Other:
- sheet Display ports: added DIGSTROBE, DIG_A0, DIG_A1, DIG_A2, DIG_A3, DOTSTROBE, SEGA1_IN, SEGA2_IN, SEGB1_IN, SEGB2_IN, SEGC1_IN, SEGC2_IN, SEGD1_IN, SEGD2_IN, SEGE1_IN, SEGE2_IN, SEGF1_IN, SEGF2_IN, SEGG1_IN, SEGG2_IN, SEGH1_IN, SEGH2_IN; removed none
- sheet GPS ports: added PPS, RX, TX; removed none
- sheet RTC ports: added BATT_SENSE, BAT_GATE_EN, RST, SCL, SDA; removed none
- moved on the sheet: R4

Commit message: board work
Parts:
- removed R1, R2: 5.1k, Resistor_SMD:R_0402_1005Metric, symbol Device:R_US
- added R17, R18, R19, R20: 100R, Resistor_SMD:R_0402_1005Metric, symbol Device:R
- added R3, R4: 5.1K, Resistor_SMD:R_0402_1005Metric, symbol Device:R
- R10: renamed from R45; footprint (none) -> Resistor_SMD:R_0402_1005Metric
- R11: renamed from R46; footprint (none) -> Resistor_SMD:R_0402_1005Metric
- renumbered C2 to C1, C6 to C10, C30 to C11, C8 to C12, C9 to C13, C10 to C14, C11 to C15, C12 to C16, C13 to C17, C14 to C18, C15 to C19, C16 to C20, C17 to C21, C18 to C22, C19 to C23, C20 to C24, C21 to C25, C1 to C3, C29 to C5, C7 to C6, C5 to C7, C31 to C8, C32 to C9, J3 to J2, Q15 to Q1, Q16 to Q2, R49 to R1, R5 to R12, R4 to R13, R7 to R14, R9 to R15, R10 to R16, R52 to R2, R50 to R5, R51 to R6, R47 to R7, R48 to R8, R3 to R9, SW3 to SW1, SW4 to SW2, SW1 to SW3, SW2 to SW4, U2 to U1, U9 to U2, U1 to U4
Connections:
- net GND: now also R3.1, R4.1
- net PPS_IN: now also R19.2
- net RUN: now also R20.2
- net UART1_RX: now also R17.2
- net UART1_TX: now also R18.2
- net at J1.A5 (CC1): now also R3.2
- net at J1.B5 (CC2): now also R4.2
- new net GPS/PPS: R19.1
- new net GPS/RX: R18.1
- new net GPS/TX: R17.1
- new net RTC/RST: R20.1

Commit message: board work
Parts:
- renumbered C4 to C1, C20 to C10, C21 to C11, C22 to C12, C23 to C13, C24 to C14, C25 to C15, C3 to C16, C13 to C17, C7 to C18, C10 to C19, C6 to C2, C1 to C20, C2 to C21, C5 to C22, C11 to C23, C8 to C24, C9 to C25, C12 to C3, C14 to C4, C15 to C5, C16 to C6, C17 to C7, C18 to C8, C19 to C9, R3 to R1, R20 to R10, R9 to R11, R13 to R12, R2 to R13, R5 to R14, R6 to R15, R7 to R16, R8 to R17, R1 to R18, R10 to R19, R4 to R2, R11 to R20, R12 to R3, R15 to R4, R16 to R5, R14 to R6, R17 to R7, R18 to R8, R19 to R9, SW3 to SW1, SW4 to SW2, SW1 to SW3, SW2 to SW4, U3 to U1, U1 to U3

Commit message: Board Rev 1.0 Release
Connections:
- net UVBUS is gone; now on net +5V: U2.5 (VBUS)
Changed lines of the file:
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@@
 	)
 	(symbol
-		(lib_id "power:VBUS")
-		(at 69.85 66.04 0)
-		(unit 1)
-		(exclude_from_sim no)
-		(in_bom yes)
-		(on_board yes)
-		(dnp no)
-		(property "Reference" "#PWR07"
-			(at 69.85 69.85 0)
-			(effects
-				(font
-					(size 1.27 1.27)
-				)
-				(hide yes)
-			)
-		)
-		(property "Value" "UVBUS"
-			(at 70.231 61.6458 0)
-			(effects
-				(font
-					(size 1.27 1.27)
-				)
-			)
-		)
-		(property "Footprint" ""
-			(at 69.85 66.04 0)
-			(effects
-				(font
-					(size 1.27 1.27)
-				)
-				(hide yes)
-			)
-		)
-		(property "Datasheet" ""
-			(at 69.85 66.04 0)
-			(effects
-				(font
-					(size 1.27 1.27)
-				)
-				(hide yes)
-			)
-		)
-		(property "Description" ""
-			(at 69.85 66.04 0)
-			(effects
-				(font
-					(size 1.27 1.27)
-				)
-				(hide yes)
-			)
-		)
-		(pin "1"
-		)
-		(instances
-			(project "precision-clock"
-				(path "/3cbd0e8e-3ba4-43b1-82ac-749e7a469b5f"
-					(reference "#PWR07")
-					(unit 1)
-				)
-			)
-		)
-	)
-	(symbol
 		(lib_id "power:+1V1")
 		(at 134.62 111.76 0)
@@
 					(unit 1)
 				)
+			)
+		)
+	)
+	(symbol
+		(lib_id "power:+5V")
+		(at 69.85 66.04 0)
+		(unit 1)
+		(exclude_from_sim no)
+		(in_bom yes)
+		(on_board yes)
+		(dnp no)
+		(fields_autoplaced yes)
+		(property "Reference" "#PWR07"
+			(at 69.85 69.85 0)
+			(effects
+				(font
+					(size 1.27 1.27)
+				)
+				(hide yes)
+			)
+		)
+		(property "Value" "+5V"
+			(at 69.85 60.96 0)
+			(effects
+				(font
+					(size 1.27 1.27)
+				)
+			)
+		)
+		(property "Footprint" ""
+			(at 69.85 66.04 0)
+			(effects
+				(font
+					(size 1.27 1.27)
+				)
+				(hide yes)
+			)
+		)
+		(property "Datasheet" ""
+			(at 69.85 66.04 0)
+			(effects
+				(font
+					(size 1.27 1.27)
+				)
+				(hide yes)
+			)
+		)
+		(property "Description" "Power symbol creates a global label with name \"+5V\""
+			(at 69.85 66.04 0)
+			(effects
+				(font
+					(size 1.27 1.27)
+				)
+				(hide yes)
+			)
+		)
+		(pin "1"
+		)
+		(instances
+			(project "precision-clock"
+				(path "/3cbd0e8e-3ba4-43b1-82ac-749e7a469b5f"
+					(reference "#PWR07")
+					(unit 1)
+				)

Commit message: BOM, CSV, and STEP exports
Parts:
- C1, C2, C6: JLCPCB PN (none) -> C32635; MFR PN (none) -> CL21B106KPQNNNE
- C10, C11, C12, C13, C14, C15, C16, C22, C23, C24, C25, C3, C5, C7, C8, C9: JLCPCB PN (none) -> C77014; MFR PN (none) -> GRM155R71E104KE14D
- C17, C18, C19, C4: JLCPCB PN (none) -> C77004; MFR PN (none) -> GRM155R61A475KEAAD
- C20, C21: JLCPCB PN (none) -> C338103; MFR PN (none) -> CGA2B2C0G1H150JT0Y0F
- J1: JLCPCB PN (none) -> C2988369; MFR PN (none) -> GT-USB-7010ASV
- L1: JLCPCB PN (none) -> C42411119; MFR PN (none) -> AOTA-B201610S3R3-101-T
- Q1, Q2: JLCPCB PN (none) -> C2900269; MFR PN (none) -> SFH 320
- R1, R2: JLCPCB PN (none) -> C105872; MFR PN (none) -> RC0402FR-075K1L
- R10, R7, R8, R9: JLCPCB PN (none) -> C106232; MFR PN (none) -> RC0402FR-07100RL
- R11, R12, R13, R14, R15, R16, R17, R6: JLCPCB PN (none) -> C106235; MFR PN (none) -> RC0402FR-071KL
- R18: JLCPCB PN (none) -> C106231; MFR PN (none) -> RC0402FR-070RL
- R19, R20: JLCPCB PN (none) -> C60490; MFR PN (none) -> RC0402FR-0710KL
- R3: JLCPCB PN (none) -> C138002; MFR PN (none) -> RC0402FR-0733RL
- R4, R5: JLCPCB PN (none) -> C138021; MFR PN (none) -> RC0402FR-0727RL
- SW1, SW2, SW3, SW4: JLCPCB PN (none) -> C2798978; MFR PN (none) -> PTS647SK38SMTR2 LFS
- U1: JLCPCB PN (none) -> C9662; MFR PN (none) -> LM1117MPX-3.3/NOPB
- U2: JLCPCB PN (none) -> C15999; MFR PN (none) -> USBLC6-2P6
- U3: JLCPCB PN (none) -> C97521; MFR PN (none) -> W25Q128JVSIQ
- U4: JLCPCB PN (none) -> C42415655; MFR PN (none) -> RP2350B
- Y1: JLCPCB PN (none) -> C20625731; MFR PN (none) -> ABM8-272-T3

Commit message: fix bom and recompress gerbers
Parts:
- SW1, SW2, SW3, SW4: JLCPCB PN C2798978 -> C2689502; MFR PN PTS647SK38SMTR2 LFS -> PTS647SM38SMTR2LFS
Changed lines of the file:
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@@
 			)
 		)
-		(property "JLCPCB PN" "C2798978 "
+		(property "JLCPCB PN" "C2689502"
 			(at 148.59 175.26 0)
 			(effects
@@
 			)
 		)
-		(property "MFR PN" "PTS647SK38SMTR2 LFS "
+		(property "MFR PN" "PTS647SM38SMTR2LFS"
 			(at 148.59 175.26 0)
 			(effects
@@
 			)
 		)
-		(property "JLCPCB PN" "C2798978 "
+		(property "JLCPCB PN" "C2689502"
 			(at 118.11 270.51 90)
 			(effects
@@
 			)
 		)
-		(property "MFR PN" "PTS647SK38SMTR2 LFS "
+		(property "MFR PN" "PTS647SM38SMTR2LFS"
 			(at 118.11 270.51 90)
 			(effects
@@
 			)
 		)
-		(property "JLCPCB PN" "C2798978 "
+		(property "JLCPCB PN" "C2689502"
 			(at 118.11 254 90)
 			(effects
@@
 			)
 		)
-		(property "MFR PN" "PTS647SK38SMTR2 LFS "
+		(property "MFR PN" "PTS647SM38SMTR2LFS"
 			(at 118.11 254 90)
 			(effects
@@
 			)
 		)
-		(property "JLCPCB PN" "C2798978 "
+		(property "JLCPCB PN" "C2689502"
 			(at 144.78 140.97 90)
 			(effects
@@
 			)
 		)
-		(property "MFR PN" "PTS647SK38SMTR2 LFS "
+		(property "MFR PN" "PTS647SM38SMTR2LFS"
 			(at 144.78 140.97 90)
 			(effects
